Commit message: new robot URDF, no front wheels yet

File: distobee_description/urdf/description.urdf.xacro (robot description, xacro)
@@ -1,96 +1,97 @@
 <?xml version="1.0"?>
 <robot xmlns:xacro="http://ros.org/wiki/xacro" name="distobee_robot">
-    <!-- Properties -->
-    <xacro:property name="base_length" value="0.5"/>
-    <xacro:property name="base_width" value="0.35"/>
-    <xacro:property name="base_height" value="0.2"/>
-    <xacro:property name="front_wheels_radius" value="0.2"/>
-    <xacro:property name="rear_wheels_radius" value="0.14"/>
-    <xacro:property name="front_wheels_width" value="0.15"/>
-    <xacro:property name="rear_wheels_width" value="0.15"/>
-    <xacro:property name="front_wheels_track" value="0.7"/>
-    <xacro:property name="rear_wheels_track" value="0.7"/>
-    <material name="red">
-      <color rgba="1 0 0 1"/>
-    </material>
-    <material name="gray">
-      <color rgba="0.5 0.5 0.5 1"/>
-    </material>
-    <!-- Base Link -->
-    <link name="base_link">
-      <visual>
-        <origin xyz="0 0 0" rpy="0 0 0"/>
-        <geometry>
-          <box size="${base_width} ${base_length} ${base_height}"/>
-        </geometry>
-        <material name="red"/>
-      </visual>
-    </link>
-    <!-- FRONT WHEELS -->
-    <!-- Front Left Wheel -->
-    <link name="front_left_wheel">
-      <visual>
-        <origin xyz="${base_length / 2} ${front_wheels_track / 2} ${front_wheels_radius}" rpy="1.5708 0 0"/>
-        <geometry>
-          <cylinder radius="${front_wheels_radius}" length="${front_wheels_width}"/>
-        </geometry>
-        <material name="gray"/>
-      </visual>
-    </link>
-    <!-- Front Right Wheel -->
-    <link name="front_right_wheel">
-      <visual>
-        <origin xyz="${base_length / 2} -${front_wheels_track / 2} ${front_wheels_radius}" rpy="1.5708 0 0"/>
-        <geometry>
-          <cylinder radius="${front_wheels_radius}" length="${front_wheels_width}"/>
-        </geometry>
-        <material name="gray"/>
-      </visual>
-    </link>
-    <!-- REAR WHEELS -->
-    <!-- Rear Left Wheel -->
-    <link name="rear_left_wheel">
-      <visual>
-        <origin xyz="-${base_length / 2} ${rear_wheels_track / 2} ${rear_wheels_radius}" rpy="1.5708 0 0"/>
-        <geometry>
-          <cylinder radius="${rear_wheels_radius}" length="${rear_wheels_width}"/>
-        </geometry>
-        <material name="gray"/>
-      </visual>
-    </link>
-    <!-- Rear Right Wheel -->
-    <link name="rear_right_wheel">
-      <visual>
-        <origin xyz="-${base_length / 2} -${rear_wheels_track / 2} ${rear_wheels_radius}" rpy="1.5708 0 0"/>
-        <geometry>
-          <cylinder radius="${rear_wheels_radius}" length="${rear_wheels_width}"/>
-        </geometry>
-        <material name="gray"/>
-      </visual>
-    </link>
-    <!-- JOINTS -->
+  <!-- ================== PROPERTIES ================== -->
+  <xacro:property name="base_length"  value="0.35"/>
+  <xacro:property name="base_width" value="0.5"/>
+  <xacro:property name="base_height" value="0.2"/>
+  <xacro:property name="distance_ground" value="0.15"/>
+  <xacro:property name="front_wheels_radius" value="0.12"/>
+  <xacro:property name="rear_wheels_radius"  value="0.2"/>
+  <xacro:property name="front_wheels_track" value="0.7"/>
+  <xacro:property name="rear_wheels_track"  value="0.7"/>
+  <!-- ================== MATERIALS ================== -->
+  <material name="red">
+    <color rgba="1 0 0 1"/>
+  </material>
+  <material name="gray">
+    <color rgba="0.5 0.5 0.5 1"/>
+  </material>
+  <!-- ================== BASE ================== -->
+  <link name="base_link">
+    <visual>
+      <origin xyz="${-base_length} ${base_width/2} ${distance_ground}" rpy="-1.5708 0 -1.5708"/>
+      <geometry>
+        <mesh filename="package://distobee_description/models/frame.obj" scale="0.001 0.001 0.001"/>
+      </geometry>
+      <material name="red"/>
+    </visual>
+  </link>
+  <!-- ================== WHEELS ================== -->
+  <!-- Rear Left Wheel -->
+  <link name="rear_left_wheel">
+    <visual>
+      <origin xyz="0 0 0" rpy="0 0 1.5708"/>
+      <geometry>
+        <mesh filename="package://distobee_description/models/rear_wheel.obj" scale="0.001 0.001 0.001"/>
+      </geometry>
+      <material name="gray"/>
+    </visual>
+  </link>
+  <!-- Rear Right Wheel -->
+  <link name="rear_right_wheel">
+    <visual>
+      <origin xyz="0 0 0" rpy="0 0 1.5708"/>
+      <geometry>
+        <mesh filename="package://distobee_description/models/rear_wheel.obj" scale="0.001 0.001 0.001"/>
+      </geometry>
+      <material name="gray"/>
+    </visual>
+  </link>
+  <!-- Front Left Wheel -->
+  <link name="front_left_wheel">
+    <visual>
+      <origin xyz="0 0 0" rpy="0 0 1.5708"/>
+      <geometry>
+        <mesh filename="package://distobee_description/models/rear_wheel.obj" scale="0.001 0.0006 0.0006"/>
+      </geometry>
+      <material name="gray"/>
+    </visual>
+  </link>
+  <!-- Front Right Wheel -->
+  <link name="front_right_wheel">
+    <visual>
+      <origin xyz="0 0 0" rpy="0 0 1.5708"/>
+      <geometry>
+        <mesh filename="package://distobee_description/models/rear_wheel.obj" scale="0.001 0.0006 0.0006"/>
+      </geometry>
+      <material name="gray"/>
+    </visual>
+  </link>
+  <!-- ================== JOINTS ================== -->
+  <!-- Rear Wheels -->
+  <joint name="rear_left_wheel_joint" type="continuous">
+    <parent link="base_link"/>
+    <child  link="rear_left_wheel"/>
+    <origin xyz="-0.2 ${rear_wheels_track/2} ${rear_wheels_radius}" rpy="0 0 0"/>
+    <axis xyz="0 1 0"/>
+  </joint>
+  <joint name="rear_right_wheel_joint" type="continuous">
+    <parent link="base_link"/>
+    <child  link="rear_right_wheel"/>
+    <origin xyz="-0.2 -${rear_wheels_track/2} ${rear_wheels_radius}" rpy="0 0 0"/>
+    <axis xyz="0 1 0"/>
+  </joint>
+  <!-- Front Wheels -->
   <joint name="front_left_wheel_joint" type="continuous">
-  <parent link="base_link"/>
-  <child link="front_left_wheel"/>
-  <origin xyz="${base_length / 2} ${front_wheels_track / 2} ${front_wheels_radius}" rpy="0 0 0"/>
-  <axis xyz="0 1 0"/>
-</joint>
-<joint name="front_right_wheel_joint" type="continuous">
-  <parent link="base_link"/>
-  <child link="front_right_wheel"/>
-  <origin xyz="${base_length / 2} -${front_wheels_track / 2} ${front_wheels_radius}" rpy="0 0 0"/>
-  <axis xyz="0 1 0"/>
-</joint>
-<joint name="rear_left_wheel_joint" type="continuous">
-  <parent link="base_link"/>
-  <child link="rear_left_wheel"/>
-  <origin xyz="-${base_length / 2} ${rear_wheels_track / 2} ${rear_wheels_radius}" rpy="0 0 0"/>
-  <axis xyz="0 1 0"/>
-</joint>
-<joint name="rear_right_wheel_joint" type="continuous">
-  <parent link="base_link"/>
-  <child link="rear_right_wheel"/>
-  <origin xyz="-${base_length / 2} -${rear_wheels_track / 2} ${rear_wheels_radius}" rpy="0 0 0"/>
-  <axis xyz="0 1 0"/>
-</joint>
+    <parent link="base_link"/>
+    <child  link="front_left_wheel"/>
+    <origin xyz="0.655 ${front_wheels_track/2} ${front_wheels_radius}" rpy="0 0 0"/>
+    <axis xyz="0 1 0"/>
+  </joint>
+  <joint name="front_right_wheel_joint" type="continuous">
+    <parent link="base_link"/>
+    <child  link="front_right_wheel"/>
+    <origin xyz="0.655 -${front_wheels_track/2} ${front_wheels_radius}" rpy="0 0 0"/>
+    <axis xyz="0 1 0"/>
+  </joint>
 </robot>
