Commit message: wip remove ros2_control

File: distobee_description/urdf/wheels.urdf.xacro (robot description, xacro)
@@ -2,6 +2,6 @@
 <robot xmlns:xacro="http://ros.org/wiki/xacro" name="distobee_robot">
   <xacro:macro name="wheels" params="base_footprint rear_wheel_radius front_wheel_radius">
-    <xacro:property name="steering_track_width" value="0.9" />
-    <xacro:property name="traction_track_width" value="0.9" />
+    <xacro:property name="steering_track_width" value="0.7" />
+    <xacro:property name="traction_track_width" value="0.7" />
     <xacro:property name="wheelbase" value="0.9" />
     <xacro:property name="steering_extension" value="0.1" />
