Commit message: major refactoring - final result is a more accurate URDF with updated ros2_control setup and gamepad steering

File: distobee_description/urdf/distobee.urdf.xacro (robot description, xacro)
@@ -1,14 +1,27 @@
 <?xml version="1.0"?>
-<!-- Basic differential drive mobile base -->
-<robot xmlns:xacro="http://www.ros.org/wiki/xacro" name="distobee_robot">
-  <xacro:arg name="prefix" default="" />
-  <xacro:arg name="use_mock_hardware" default="false" />
-  <xacro:include filename="$(find distobee_description)/urdf/distobee_description.urdf.xacro" />
-  <!-- Import Rviz colors -->
-  <!--<xacro:include filename="$(find odrive_botwheel_explorer)/urdf/diffbot.materials.xacro" />-->
-  <!-- Import ros2_control description -->
-  <xacro:include filename="$(find distobee_description)/urdf/distobee.ros2_control.xacro" />
-  <xacro:diffbot prefix="$(arg prefix)" />
-  <xacro:distobee_ros2_control
-    name="distobee" prefix="$(arg prefix)" use_mock_hardware="$(arg use_mock_hardware)"/>
+<robot xmlns:xacro="http://www.ros.org/wiki/xacro" name="distobee">
+  <material name="white">
+    <color rgba="0.8 0.8 0.8 1" />
+  </material>
+  <!-- https://www.ros.org/reps/rep-0120.html -->
+  <link name="base_footprint" />
+  <link name="base_link">
+    <visual>
+      <geometry>
+        <mesh filename="package://distobee_description/stl/body.stl" />
+      </geometry>
+      <material name="white" />
+    </visual>
+  </link>
+  <joint name="base_joint" type="fixed">
+    <origin xyz="-0.2 0 0.15" />
+    <parent link="base_footprint" />
+    <child link="base_link" />
+  </joint>
+  <!-- wheels -->
+  <xacro:include filename="$(find distobee_description)/urdf/wheels.urdf.xacro" />
+  <xacro:wheels base_footprint="base_footprint" wheel_radius="0.2" />
+  <!-- ros2_control -->
+  <xacro:include filename="$(find distobee_description)/urdf/ros2_control.urdf.xacro" />
+  <xacro:ros2_control />
 </robot>

Commit message: scale down front wheels

File: distobee_description/urdf/distobee.urdf.xacro (robot description, xacro)
@@ -21,5 +21,5 @@
   <!-- wheels -->
   <xacro:include filename="$(find distobee_description)/urdf/wheels.urdf.xacro" />
-  <xacro:wheels base_footprint="base_footprint" wheel_radius="0.2" />
+  <xacro:wheels base_footprint="base_footprint" rear_wheel_radius="0.2" front_wheel_radius="0.14" />
   <!-- ros2_control -->
   <xacro:include filename="$(find distobee_description)/urdf/ros2_control.urdf.xacro" />

File: distobee_description/urdf/wheels.urdf.xacro (robot description, xacro)
@@ -1,9 +1,12 @@
 <?xml version="1.0"?>
 <robot xmlns:xacro="http://ros.org/wiki/xacro" name="distobee_robot">
-  <xacro:macro name="wheels" params="base_footprint wheel_radius">
+  <xacro:macro name="wheels" params="base_footprint rear_wheel_radius front_wheel_radius">
     <xacro:property name="steering_track_width" value="0.9" />
     <xacro:property name="traction_track_width" value="0.9" />
     <xacro:property name="wheelbase" value="0.9" />
     <xacro:property name="steering_extension" value="0.1" />
+    <!-- FIXME: Temporary reuse of a scaled down rear wheel mesh for the front wheels. Please remove
+    this scaling and provide a separate mesh once it's ready. -->
+    <xacro:property name="front_wheel_scale" value="${front_wheel_radius / rear_wheel_radius}" />
     <link name="wheel_bl_link">
       <visual>
@@ -18,5 +21,5 @@
       <parent link="${base_footprint}" />
       <child link="wheel_bl_link" />
-      <origin xyz="${-wheelbase/2} ${traction_track_width/2} ${wheel_radius}" rpy="0 0 0" />
+      <origin xyz="${-wheelbase/2} ${traction_track_width/2} ${rear_wheel_radius}" rpy="0 0 0" />
       <axis xyz="0 1 0" />
     </joint>
@@ -33,5 +36,5 @@
       <parent link="${base_footprint}" />
       <child link="wheel_br_link" />
-      <origin xyz="${-wheelbase/2} ${-traction_track_width/2} ${wheel_radius}" rpy="0 0 0" />
+      <origin xyz="${-wheelbase/2} ${-traction_track_width/2} ${rear_wheel_radius}" rpy="0 0 0" />
       <axis xyz="0 1 0" />
     </joint>
@@ -40,5 +43,7 @@
       <parent link="${base_footprint}" />
       <child link="turn_fl_link" />
-      <origin xyz="${wheelbase/2} ${steering_track_width/2 - steering_extension} ${wheel_radius}" rpy="0 0 0" />
+      <origin
+        xyz="${wheelbase/2} ${steering_track_width/2 - steering_extension} ${front_wheel_radius}"
+        rpy="0 0 0" />
       <axis xyz="0 0 1" />
       <limit lower="-0.3" upper="0.3" effort="100.0" velocity="1.0" />
@@ -48,5 +53,6 @@
         <origin xyz="0 0 0" rpy="0 0 0" />
         <geometry>
-          <mesh filename="package://distobee_description/stl/rear_wheel.stl" />
+          <mesh filename="package://distobee_description/stl/rear_wheel.stl"
+            scale="${front_wheel_scale} ${front_wheel_scale} ${front_wheel_scale}" />
         </geometry>
         <material name="white" />
@@ -63,5 +69,7 @@
       <parent link="${base_footprint}" />
       <child link="turn_fr_link" />
-      <origin xyz="${wheelbase/2} ${-steering_track_width/2 + steering_extension} ${wheel_radius}" rpy="0 0 0" />
+      <origin
+        xyz="${wheelbase/2} ${-steering_track_width/2 + steering_extension} ${front_wheel_radius}"
+        rpy="0 0 0" />
       <axis xyz="0 0 1" />
       <limit lower="-0.3" upper="0.3" effort="100.0" velocity="1.0" />
@@ -71,5 +79,6 @@
         <origin xyz="0 0 0" rpy="0 0 0" />
         <geometry>
-          <mesh filename="package://distobee_description/stl/rear_wheel.stl" />
+          <mesh filename="package://distobee_description/stl/rear_wheel.stl"
+            scale="${front_wheel_scale} ${front_wheel_scale} ${front_wheel_scale}" />
         </geometry>
         <material name="white" />

Commit message: better wheels measurements

File: distobee_description/urdf/distobee.urdf.xacro (robot description, xacro)
@@ -21,5 +21,5 @@
   <!-- wheels -->
   <xacro:include filename="$(find distobee_description)/urdf/wheels.urdf.xacro" />
-  <xacro:wheels base_footprint="base_footprint" rear_wheel_radius="0.2" front_wheel_radius="0.14" />
+  <xacro:wheels base_footprint="base_footprint" rear_wheel_radius="0.2" front_wheel_radius="0.125" />
   <!-- ros2_control -->
   <xacro:include filename="$(find distobee_description)/urdf/ros2_control.urdf.xacro" />

File: distobee_description/urdf/wheels.urdf.xacro (robot description, xacro)
@@ -2,8 +2,8 @@
 <robot xmlns:xacro="http://ros.org/wiki/xacro" name="distobee_robot">
   <xacro:macro name="wheels" params="base_footprint rear_wheel_radius front_wheel_radius">
-    <xacro:property name="steering_track_width" value="0.7" />
+    <xacro:property name="steering_track_width" value="0.6" />
     <xacro:property name="traction_track_width" value="0.7" />
     <xacro:property name="wheelbase" value="0.9" />
-    <xacro:property name="steering_extension" value="0.1" />
+    <xacro:property name="steering_extension" value="0.0" />
     <!-- FIXME: Temporary reuse of a scaled down rear wheel mesh for the front wheels. Please remove
     this scaling and provide a separate mesh once it's ready. -->
